Commit message: controller added

File: src/aura_description/urdf/aura_base.xacro (robot description, xacro)
@@ -1,7 +1,5 @@
 <?xml version="1.0" ?>
 <robot name="aura" xmlns:xacro="http://www.ros.org/wiki/xacro">
-  <!-- Start GZ or Ignition depending on ROS 2 Version -->
   <xacro:arg name="is_ignition" default="true"/>
-  <!-- Load Simulated or Real Hardware Interfaces -->
   <xacro:arg name="is_sim" default="true"/>
   <link name="base_footprint" />
@@ -70,12 +68,12 @@
     </visual>
     <collision>
-      <origin xyz="0.12 0.0 -0.015" rpy="0 0 0"/>
-      <geometry>
-        <mesh filename="package://aura_description/meshes/back_castor.stl" scale="0.001 0.001 0.001"/>
-      </geometry>
-    </collision>
-  </link>
-  <joint name="base_back_castor_joint" type="fixed">
-    <origin xyz="-0.12 0.0 0.015" rpy="0 0 0"/>
+      <origin xyz="0.0 0.0 0.0" rpy="0.0 0.0 0.0"/>
+      <geometry>
+        <sphere radius="0.015"/>
+      </geometry>
+    </collision>
+  </link>
+  <joint name="back_castor_joint" type="fixed">
+    <origin xyz="-0.12 0.0 0.0151" rpy="0 0 0"/>
     <parent link="base_link"/>
     <child link="back_castor"/>
@@ -83,5 +81,5 @@
   <link name="front_castor">
     <inertial>
-      <origin xyz="-0.12 0.0 -0.015" rpy="0 0 0"/>
+      <origin xyz="-0.12 0.0 -0.15" rpy="0 0 0"/>
       <mass value="0.030997748883593468"/>
       <inertia ixx="3e-06" iyy="3e-06" izz="5e-06" ixy="-0.0" iyz="0.0" ixz="0.0"/>
@@ -95,12 +93,13 @@
     </visual>
     <collision>
-      <origin xyz="-0.12 0.0 -0.015" rpy="0 0 0"/>
-      <geometry>
-        <mesh filename="package://aura_description/meshes/front_castor.stl" scale="0.001 0.001 0.001"/>
-      </geometry>
-    </collision>
-  </link>
-  <joint name="base_front_castor_joint" type="fixed">
-    <origin xyz="0.12 0.0 0.015" rpy="0 0 0"/>
+     <!-- <origin xyz="-0.12 0.0 -0.015" rpy="0 0 0"/> -->
+     <origin xyz="0.0 0.0 0.0" rpy="0.0 0.0 0.0"/>
+      <geometry>
+        <sphere radius="0.015"/>
+      </geometry>
+    </collision>
+  </link>
+  <joint name="front_castor_joint" type="fixed">
+    <origin xyz="0.12 0.0 0.0151" rpy="0 0 0"/>
     <parent link="base_link"/>
     <child link="front_castor"/>
@@ -109,6 +108,6 @@
     <inertial>
       <origin xyz="-4.135866654458078e-07 -0.022655023372287864 -6.624769580132472e-08" rpy="0 0 0"/>
-      <mass value="0.2385962385065163"/>
-      <inertia ixx="0.000155" iyy="0.000225" izz="0.000155" ixy="0.0" iyz="-0.0" ixz="0.0"/>
+      <mass value="2.2063738184473554"/>
+      <inertia ixx="0.00143" iyy="0.002082" izz="0.00143" ixy="0.0" iyz="-0.0" ixz="-0.0"/>
     </inertial>
     <visual>
@@ -126,5 +125,5 @@
     </collision>
   </link>
-  <joint name="wall_right_wheel_joint" type="continuous">
+  <joint name="right_wheel_joint" type="continuous">
     <origin xyz="-8.9e-05 -0.128 0.010091" rpy="0 0 0"/>
     <parent link="wall"/>
@@ -134,5 +133,5 @@
   <link name="left_wheel">
     <inertial>
-      <origin xyz="-4.135866654364159e-07 0.022655023372287864 -6.62476958360192e-08" rpy="0 0 0"/>
+      <origin xyz="-4.135866654458078e-07 0.022655023372287864 -6.624769580132472e-08" rpy="0 0 0"/>
       <mass value="2.2063738184473554"/>
       <inertia ixx="0.00143" iyy="0.002082" izz="0.00143" ixy="0.0" iyz="-0.0" ixz="-0.0"/>
@@ -152,5 +151,5 @@
     </collision>
   </link>
-  <joint name="wall_left_wheel_joint" type="continuous">
+  <joint name="left_wheel_joint" type="continuous">
     <origin xyz="-8.9e-05 0.128 0.010091" rpy="0 0 0"/>
     <parent link="wall"/>

File: src/aura_description/urdf/aura_gazebo.xacro (robot description, xacro)
@@ -39,7 +39,6 @@
     <gazebo>
         <!-- ROS 2 Humble -->
-        <xacro:if value="$(arg is_ignition)">
         <plugin filename="ign_ros2_control-system" name="ign_ros2_control::IgnitionROS2ControlPlugin">
-            <parameters>$(find bumperbot_controller)/config/bumperbot_controllers.yaml</parameters>
+            <parameters>$(find aura_controller)/config/aura_controllers.yaml</parameters>
         </plugin>
         <plugin filename="ignition-gazebo-imu-system" name="ignition::gazebo::systems::Imu">
@@ -48,16 +47,4 @@
             <render_engine>ogre2</render_engine>
         </plugin>
-        </xacro:if>
-        <!-- ROS 2 Iron or above -->
-        <xacro:unless value="$(arg is_ignition)">
-        <plugin filename="gz_ros2_control-system" name="gz_ros2_control::GazeboSimROS2ControlPlugin">
-            <parameters>$(find bumperbot_controller)/config/bumperbot_controllers.yaml</parameters>
-        </plugin>
-        <plugin filename="gz-sim-imu-system" name="gz::sim::systems::Imu">
-        </plugin>
-        <plugin filename="gz-sim-sensors-system" name="gz::sim::systems::Sensors">
-            <render_engine>ogre2</render_engine>
-        </plugin>
-        </xacro:unless>
     </gazebo>
     <!-- Aura Sensors -->

File: src/aura_description/urdf/aura_ros2control.xacro (robot description, xacro)
@@ -25,5 +25,5 @@
         </xacro:unless>
         <!-- ros2_control Common Interfaces -->
-        <joint name="wall_right_wheel_joint">
+        <joint name="right_wheel_joint">
             <command_interface name="velocity">
               <param name="min">-1</param>
@@ -33,5 +33,5 @@
             <state_interface name="velocity" />
         </joint>
-        <joint name="wall_left_wheel_joint">
+        <joint name="left_wheel_joint">
             <command_interface name="velocity">
               <param name="min">-1</param>

Commit message: Joystick Teleop Done

File: src/aura_description/urdf/aura_base.xacro (robot description, xacro)
@@ -129,5 +129,5 @@
     <parent link="wall"/>
     <child link="right_wheel"/>
-    <axis xyz="-0.0 -1.0 0.0"/>
+    <axis xyz="-0.0 1.0 0.0"/>
   </joint>
   <link name="left_wheel">
@@ -155,5 +155,5 @@
     <parent link="wall"/>
     <child link="left_wheel"/>
-    <axis xyz="0.0 -1.0 -0.0"/>
+    <axis xyz="0.0 1.0 -0.0"/>
   </joint>
   <link name="imu_link">
