Commit message: sensor plugins added and tested

File: src/aura_description/urdf/aura.urdf.xacro (robot description, xacro)
@@ -1,7 +1,7 @@
 <?xml version="1.0"?>
 <robot name="aura" xmlns:xacro="http://www.ros.org/wiki/xacro">
-    <xacro:include filename="$(find aura_description)/urdf/aura_materials.xacro" />
-    <xacro:include filename="$(find aura_description)/urdf/aura_base.xacro" />
-  <!-- <xacro:include filename="$(find aura_description)/urdf/aura_ros2control.xacro" />
-  <xacro:include filename="$(find aura_description)/urdf/aura_gazebo.xacro" /> -->
+  <xacro:include filename="$(find aura_description)/urdf/aura_materials.xacro" />
+  <xacro:include filename="$(find aura_description)/urdf/aura_base.xacro" />
+  <xacro:include filename="$(find aura_description)/urdf/aura_gazebo.xacro" />
+  <xacro:include filename="$(find aura_description)/urdf/aura_ros2control.xacro" />
 </robot>

File: src/aura_description/urdf/aura_base.xacro (robot description, xacro)
@@ -1,4 +1,8 @@
 <?xml version="1.0" ?>
 <robot name="aura" xmlns:xacro="http://www.ros.org/wiki/xacro">
+  <!-- Start GZ or Ignition depending on ROS 2 Version -->
+  <xacro:arg name="is_ignition" default="true"/>
+  <!-- Load Simulated or Real Hardware Interfaces -->
+  <xacro:arg name="is_sim" default="true"/>
   <link name="base_footprint" />
   <link name="base_link">
@@ -13,5 +17,5 @@
         <mesh filename="package://aura_description/meshes/base_link.stl" scale="0.001 0.001 0.001"/>
       </geometry>
-      <material name="silver"/>
+      <material name="matte_brown"/>
     </visual>
     <collision>
@@ -47,5 +51,5 @@
     </collision>
   </link>
-  <joint name="base_wall" type="fixed">
+  <joint name="base_wall_joint" type="fixed">
     <origin xyz="0.0 0.0 0.033" rpy="0 0 0"/>
     <parent link="base_link"/>
@@ -72,5 +76,5 @@
     </collision>
   </link>
-  <joint name="base_back_castor" type="fixed">
+  <joint name="base_back_castor_joint" type="fixed">
     <origin xyz="-0.12 0.0 0.015" rpy="0 0 0"/>
     <parent link="base_link"/>
@@ -97,5 +101,5 @@
     </collision>
   </link>
-  <joint name="base_front_castor" type="fixed">
+  <joint name="base_front_castor_joint" type="fixed">
     <origin xyz="0.12 0.0 0.015" rpy="0 0 0"/>
     <parent link="base_link"/>
@@ -122,5 +126,5 @@
     </collision>
   </link>
-  <joint name="wall_right_wheel" type="continuous">
+  <joint name="wall_right_wheel_joint" type="continuous">
     <origin xyz="-8.9e-05 -0.128 0.010091" rpy="0 0 0"/>
     <parent link="wall"/>
@@ -148,5 +152,5 @@
     </collision>
   </link>
-  <joint name="wall_left_wheel" type="continuous">
+  <joint name="wall_left_wheel_joint" type="continuous">
     <origin xyz="-8.9e-05 0.128 0.010091" rpy="0 0 0"/>
     <parent link="wall"/>
@@ -154,5 +158,5 @@
     <axis xyz="0.0 -1.0 -0.0"/>
   </joint>
-  <link name="imu">
+  <link name="imu_link">
     <inertial>
       <origin xyz="0.0 0.0 -0.033" rpy="0 0 0"/>
@@ -174,8 +178,8 @@
     </collision>
   </link>
-  <joint name="base_imu" type="fixed">
+  <joint name="base_imu_joint" type="fixed">
     <origin xyz="0.0 0.0 0.033" rpy="0 0 0"/>
     <parent link="base_link"/>
-    <child link="imu"/>
+    <child link="imu_link"/>
   </joint>
   <link name="top_plate">
@@ -199,10 +203,10 @@
     </collision>
   </link>
-  <joint name="base_top_plate" type="fixed">
+  <joint name="base_top_plate_joint" type="fixed">
     <origin xyz="0.0 0.0 0.1" rpy="0 0 0"/>
     <parent link="base_link"/>
     <child link="top_plate"/>
   </joint>
-  <link name="camera">
+  <link name="camera_link">
     <inertial>
      <origin xyz="-0.15 0.0 -0.118" rpy="0 0 0"/>
@@ -224,10 +228,16 @@
     </collision>
   </link>
-  <joint name="base_link_camera" type="fixed">
+  <joint name="base_camera_joint" type="fixed">
     <origin xyz="0.15 0.0 0.118" rpy="0 0 0"/>
     <parent link="base_link"/>
-    <child link="camera"/>
-  </joint>
-  <link name="lidar">
+    <child link="camera_link"/>
+  </joint>
+    <link name="camera_link_optical" />
+    <joint name="camera_optical_joint" type="fixed">
+        <parent link="camera_link"/>
+        <child link="camera_link_optical"/>
+        <origin xyz="0 0 0" rpy="${-pi/2} 0 ${-pi/2}"/>
+    </joint>
+  <link name="lidar_link">
     <inertial>
       <origin xyz="0.0 0.0 -0.16" rpy="0 0 0"/>
@@ -249,8 +259,8 @@
     </collision>
   </link>
-  <joint name="base_lidar" type="fixed">
+  <joint name="base_lidar_joint" type="fixed">
     <origin xyz="0.0 0.0 0.16" rpy="0 0 0"/>
     <parent link="base_link"/>
-    <child link="lidar"/>
+    <child link="lidar_link"/>
   </joint>
 </robot>

File: src/aura_description/urdf/aura_materials.xacro (robot description, xacro)
@@ -1,4 +1,5 @@
 <?xml version="1.0" ?>
 <robot name="aura" xmlns:xacro="http://www.ros.org/wiki/xacro">
+    <!-- Rviz Materials -->
     <!-- Silver material -->
     <material name="silver">

Commit message: URDF of Arm added Basic

File: src/aura_description/urdf/aura.urdf.xacro (robot description, xacro)
@@ -3,4 +3,5 @@
   <xacro:include filename="$(find aura_description)/urdf/aura_materials.xacro" />
   <xacro:include filename="$(find aura_description)/urdf/aura_base.xacro" />
+  <!-- <xacro:include filename="$(find aura_description)/urdf/aura_arm.xacro" /> -->
   <xacro:include filename="$(find aura_description)/urdf/aura_gazebo.xacro" />
   <xacro:include filename="$(find aura_description)/urdf/aura_ros2control.xacro" />

File: src/aura_description/urdf/aura_materials.xacro (robot description, xacro)
@@ -22,3 +22,30 @@
         <color rgba="1.000 0.980 0.850 1.000"/>
     </material>
+    <xacro:macro name="box_inertia" params="m l w h xyz rpy">
+        <inertial>
+            <origin xyz="${xyz}" rpy="${rpy}" />
+            <mass value="${m}" />
+            <inertia ixx="${(m/12) * (h*h + l*l)}" ixy="0" ixz="0"
+                     iyy="${(m/12) * (w*w + l*l)}" iyz="0"
+                     izz="${(m/12) * (w*w + h*h)}" />
+        </inertial>
+    </xacro:macro>
+    <xacro:macro name="cylinder_inertia" params="m r h xyz rpy">
+        <inertial>
+            <origin xyz="${xyz}" rpy="${rpy}" />
+            <mass value="${m}" />
+            <inertia ixx="${(m/12) * (3*r*r + h*h)}" ixy="0" ixz="0"
+                     iyy="${(m/12) * (3*r*r + h*h)}" iyz="0"
+                     izz="${(m/2) * (r*r)}" />
+        </inertial>
+    </xacro:macro>
+    <!-- <xacro:macro name="sphere_inertia" params="m r xyz rpy">
+        <inertial>
+            <origin xyz="${xyz}" rpy="${rpy}" />
+            <mass value="${m}" />
+            <inertia ixx="${((2*m)/5) * (r*r)}" ixy="0" ixz="0"
+                     iyy="${((2*m)/5) * (r*r)}" iyz="0"
+                     izz="${((2*m)/5) * (r*r)}" />
+        </inertial>
+    </xacro:macro> -->
 </robot>

Commit message: arm controllers added

File: src/aura_description/urdf/aura.urdf.xacro (robot description, xacro)
@@ -3,5 +3,5 @@
   <xacro:include filename="$(find aura_description)/urdf/aura_materials.xacro" />
   <xacro:include filename="$(find aura_description)/urdf/aura_base.xacro" />
-  <!-- <xacro:include filename="$(find aura_description)/urdf/aura_arm.xacro" /> -->
+  <xacro:include filename="$(find aura_description)/urdf/aura_arm.xacro" />
   <xacro:include filename="$(find aura_description)/urdf/aura_gazebo.xacro" />
   <xacro:include filename="$(find aura_description)/urdf/aura_ros2control.xacro" />

File: src/aura_description/urdf/aura_arm.xacro (robot description, xacro)
@@ -40,10 +40,10 @@
         </collision>
     </link>
-    <joint name="arm_base_joint" type="revolute">
+    <joint name="joint_1" type="revolute">
         <origin xyz="0.0 0.0 0.100" rpy="0.0 0.0 0.0"/>
         <parent link="arm_stand"/>
         <child link="arm_base"/>
         <axis xyz="0 0 1"/>
-        <limit lower="-3.14" upper="3.14" effort="10.0" velocity="10.0"/>
+        <limit lower="-3.14" upper="3.14" effort="30.0" velocity="10.0"/>
     </joint>
     <link name="arm_lower">
@@ -64,10 +64,10 @@
         </collision>
     </link>
-    <joint name="arm_lower_joint" type="revolute">
+    <joint name="joint_2" type="revolute">
         <origin xyz="0.0 0.0 0.04" rpy="0.0 0.0 0.0"/>
         <parent link="arm_base"/>
         <child link="arm_lower"/>
         <axis xyz="0 1 0"/>
-        <limit lower="-1.57" upper="1.57" effort="10.0" velocity="10.0"/>
+        <limit lower="-1.57" upper="1.57" effort="30.0" velocity="10.0"/>
     </joint>
     <link name="arm_upper">
@@ -88,16 +88,16 @@
         </collision>
     </link>
-    <joint name="arm_upper_joint" type="revolute">
+    <joint name="joint_3" type="revolute">
         <origin xyz="0.0 0.0 0.14" rpy="0.0 0.0 0.0"/>
         <parent link="arm_lower"/>
         <child link="arm_upper"/>
         <axis xyz="0 1 0"/>
-        <limit lower="-2.5" upper="2.5" effort="10.0" velocity="10.0"/>
+        <limit lower="-2.5" upper="2.5" effort="30.0" velocity="10.0"/>
     </joint>
     <link name="end_effector">
-        <xacro:box_inertia m="0.100" l="0.03" w="0.03" h="0.012"
-                                    xyz="0 0 -0.55" rpy="0 0 0" />
+        <xacro:box_inertia m="0.150" l="0.04" w="0.04" h="0.03"
+                                    xyz="0 0 -0.565" rpy="0 0 0" />
         <visual>
-            <origin xyz="0 0 -0.55" rpy="0 0 0"/>
+            <origin xyz="0 0 -0.565" rpy="0 0 0"/>
             <geometry>
                 <mesh filename="package://aura_description/meshes/end_effector.stl" scale="0.001 0.001 0.001"/>
@@ -106,5 +106,5 @@
         </visual>
         <collision>
-            <origin xyz="0 0 -0.55" rpy="0 0 0"/>
+            <origin xyz="0 0 -0.565" rpy="0 0 0"/>
             <geometry>
                 <mesh filename="package://aura_description/meshes/end_effector.stl" scale="0.001 0.001 0.001"/>
@@ -112,8 +112,10 @@
         </collision>
     </link>
-    <joint name="end_effector_joint" type="fixed">
+    <joint name="joint_4" type="revolute">
         <origin xyz="0.0 0.0 0.16" rpy="0.0 0.0 0.0"/>
         <parent link="arm_upper"/>
         <child link="end_effector"/>
+        <axis xyz="0 1 0"/>
+        <limit lower="-1.57" upper="1.57" effort="30.0" velocity="10.0"/>
     </joint>
 </robot>

File: src/aura_description/urdf/aura_ros2control.xacro (robot description, xacro)
@@ -2,4 +2,5 @@
 <robot name="aura" xmlns:xacro="http://www.ros.org/wiki/xacro">
     <ros2_control name="RobotSystem" type="system">
+        <xacro:property name="PI" value="3.14159265359" />
         <!-- ros2_control Gazebo -->
         <xacro:if value="$(arg is_sim)">
@@ -41,4 +42,32 @@
             <state_interface name="velocity" />
         </joint>
+        <joint name="joint_1">
+            <command_interface name="position">
+            <param name="min">-${PI / 2}</param>
+            <param name="max">${PI / 2}</param>
+            </command_interface>
+            <state_interface name="position"/>
+        </joint>
+        <joint name="joint_2">
+            <command_interface name="position">
+            <param name="min">-${PI / 2}</param>
+            <param name="max">${PI / 2}</param>
+            </command_interface>
+            <state_interface name="position"/>
+        </joint>
+        <joint name="joint_3">
+            <command_interface name="position">
+            <param name="min">-${PI / 2}</param>
+            <param name="max">${PI / 2}</param>
+            </command_interface>
+            <state_interface name="position"/>
+        </joint>
+        <joint name="joint_4">
+            <command_interface name="position">
+            <param name="min">-${PI / 2}</param>
+            <param name="max">${PI / 2}</param>
+            </command_interface>
+            <state_interface name="position"/>
+        </joint>
     </ros2_control>
 </robot>
