Commit message: Obstacle Avoidance Added in Task Script

File: src/aura_description/urdf/aura_arm.xacro (robot description, xacro)
@@ -119,3 +119,25 @@
         <limit lower="-1.57" upper="1.57" effort="30.0" velocity="10.0"/>
     </joint>
+    <!-- Suction Gripper -->
+    <!-- <link name="suction_link">
+        <xacro:box_inertia m="0.150" l="0.04" w="0.04" h="0.03"
+                                    xyz="0 0 -0.565" rpy="0 0 0" />
+        <visual>
+            <origin xyz="0 0 -0.565" rpy="0 0 0"/>
+            <geometry>
+                <mesh filename="package://aura_description/meshes/end_effector.stl" scale="0.001 0.001 0.001"/>
+            </geometry>
+            <material name="matte_brown"/>
+        </visual>
+        <collision>
+            <origin xyz="0 0 -0.565" rpy="0 0 0"/>
+            <geometry>
+                <mesh filename="package://aura_description/meshes/end_effector.stl" scale="0.001 0.001 0.001"/>
+            </geometry>
+        </collision>
+    </link>
+    <joint name="end_effector_suction_joint" type="fixed">
+        <parent link="end_effector"/>
+        <child link="suction_link"/>
+    </joint> -->
 </robot>

File: src/aura_description/urdf/aura_gazebo.xacro (robot description, xacro)
@@ -47,4 +47,7 @@
             <render_engine>ogre2</render_engine>
         </plugin>
+        <!-- <gazebo>
+            <plugin filename="libignition-gazebo-link-attacher-system.so" name="ignition::gazebo::systems::LinkAttacher"/>
+        </gazebo> -->
     </gazebo>
     <!-- Aura Sensors -->
