Commit message: Red Bar Arm Working

File: install/aura_description/share/aura_description/urdf/aura_arm.xacro (robot description, xacro)
@@ -18,5 +18,5 @@
         </collision>
     </link>
-    <joint name="arm_stand_joint" type="fixed">
+    <joint name="virtual_joint" type="fixed">
         <origin xyz="0.0 0.0 0.0" rpy="0.0 0.0 0.0"/>
         <parent link="top_plate"/>
