Commit message: Both Color Bars Woking and Auto Docking

File: install/aura_description/share/aura_description/urdf/aura.urdf.xacro (robot description, xacro)
@@ -1,8 +1 @@
-<?xml version="1.0"?>
-<robot name="aura" xmlns:xacro="http://www.ros.org/wiki/xacro">
-  <xacro:include filename="$(find aura_description)/urdf/aura_materials.xacro" />
-  <xacro:include filename="$(find aura_description)/urdf/aura_base.xacro" />
-  <xacro:include filename="$(find aura_description)/urdf/aura_arm.xacro" />
-  <xacro:include filename="$(find aura_description)/urdf/aura_gazebo.xacro" />
-  <xacro:include filename="$(find aura_description)/urdf/aura_ros2control.xacro" />
-</robot>
+/home/utk/aura_ws/src/aura_description/urdf/aura.urdf.xacro

File: install/aura_description/share/aura_description/urdf/aura_arm.xacro (robot description, xacro)
@@ -1,198 +1 @@
-<?xml version="1.0"?>
-<robot name="aura" xmlns:xacro="http://www.ros.org/wiki/xacro">
-    <link name="arm_stand">
-        <xacro:box_inertia m="0.500" l="0.10" w="0.10" h="0.08"
-                                    xyz="0 0 -0.100" rpy="0 0 0" />
-        <visual>
-            <origin xyz="0 0 -0.100" rpy="0 0 0"/>
-            <geometry>
-                <mesh filename="package://aura_description/meshes/arm_stand.stl" scale="0.001 0.001 0.001"/>
-            </geometry>
-            <material name="mud_yellow"/>
-        </visual>
-        <collision>
-            <origin xyz="0 0 -0.100" rpy="0 0 0"/>
-            <geometry>
-                <mesh filename="package://aura_description/meshes/arm_stand.stl" scale="0.001 0.001 0.001"/>
-            </geometry>
-        </collision>
-    </link>
-    <joint name="virtual_joint" type="fixed">
-        <origin xyz="0.0 0.0 0.0" rpy="0.0 0.0 0.0"/>
-        <parent link="top_plate"/>
-        <child link="arm_stand"/>
-    </joint>
-    <link name="arm_base">
-        <xacro:box_inertia m="0.200" l="0.05" w="0.05" h="0.03"
-                                    xyz="0 0 -0.200" rpy="0 0 0" />
-        <visual>
-            <origin xyz="0 0 -0.200" rpy="0 0 0"/>
-            <geometry>
-                <mesh filename="package://aura_description/meshes/arm_base.stl" scale="0.001 0.001 0.001"/>
-            </geometry>
-            <material name="silver"/>
-        </visual>
-        <collision>
-            <origin xyz="0 0 -0.200" rpy="0 0 0"/>
-            <geometry>
-                <mesh filename="package://aura_description/meshes/arm_base.stl" scale="0.001 0.001 0.001"/>
-            </geometry>
-        </collision>
-    </link>
-    <joint name="joint_1" type="revolute">
-        <origin xyz="0.0 0.0 0.100" rpy="0.0 0.0 0.0"/>
-        <parent link="arm_stand"/>
-        <child link="arm_base"/>
-        <axis xyz="0 0 1"/>
-        <limit lower="-3.14" upper="3.14" effort="30.0" velocity="10.0"/>
-    </joint>
-    <link name="arm_lower">
-        <xacro:cylinder_inertia m="0.500" r="0.02" h="0.15"
-                            xyz="0 0 -0.24" rpy="0 0 0" />
-        <visual>
-            <origin xyz="0 0 -0.24" rpy="0 0 0"/>
-            <geometry>
-                <mesh filename="package://aura_description/meshes/arm_lower.stl" scale="0.001 0.001 0.001"/>
-            </geometry>
-            <material name="silver"/>
-        </visual>
-        <collision>
-            <origin xyz="0 0 -0.24" rpy="0 0 0"/>
-            <geometry>
-                <mesh filename="package://aura_description/meshes/arm_lower.stl" scale="0.001 0.001 0.001"/>
-            </geometry>
-        </collision>
-    </link>
-    <joint name="joint_2" type="revolute">
-        <origin xyz="0.0 0.0 0.04" rpy="0.0 0.0 0.0"/>
-        <parent link="arm_base"/>
-        <child link="arm_lower"/>
-        <axis xyz="0 1 0"/>
-        <limit lower="-1.57" upper="1.57" effort="30.0" velocity="10.0"/>
-    </joint>
-    <link name="arm_upper">
-        <xacro:cylinder_inertia m="0.500" r="0.02" h="0.15"
-                            xyz="0 0 -0.39" rpy="0 0 0" />
-        <visual>
-            <origin xyz="0 0 -0.39" rpy="0 0 0"/>
-            <geometry>
-                <mesh filename="package://aura_description/meshes/arm_upper.stl" scale="0.001 0.001 0.001"/>
-            </geometry>
-            <material name="silver"/>
-        </visual>
-        <collision>
-            <origin xyz="0 0 -0.39" rpy="0 0 0"/>
-            <geometry>
-                <mesh filename="package://aura_description/meshes/arm_upper.stl" scale="0.001 0.001 0.001"/>
-            </geometry>
-        </collision>
-    </link>
-    <joint name="joint_3" type="revolute">
-        <origin xyz="0.0 0.0 0.14" rpy="0.0 0.0 0.0"/>
-        <parent link="arm_lower"/>
-        <child link="arm_upper"/>
-        <axis xyz="0 1 0"/>
-        <limit lower="-2.5" upper="2.5" effort="30.0" velocity="10.0"/>
-    </joint>
-    <link name="claw_support">
-        <xacro:box_inertia m="0.150" l="0.04" w="0.04" h="0.03"
-                                    xyz="0 0 -0.565" rpy="0 0 0" />
-        <visual>
-            <origin xyz="0 0 -0.565" rpy="0 0 0"/>
-            <geometry>
-                <mesh filename="package://aura_description/meshes/end_effector.stl" scale="0.001 0.001 0.001"/>
-            </geometry>
-            <material name="matte_brown"/>
-        </visual>
-        <collision>
-            <origin xyz="0 0 -0.565" rpy="0 0 0"/>
-            <geometry>
-                <mesh filename="package://aura_description/meshes/end_effector.stl" scale="0.001 0.001 0.001"/>
-            </geometry>
-        </collision>
-    </link>
-    <joint name="joint_4" type="revolute">
-        <origin xyz="0.0 0.0 0.16" rpy="0.0 0.0 0.0"/>
-        <parent link="arm_upper"/>
-        <child link="claw_support"/>
-        <axis xyz="0 1 0"/>
-        <limit lower="-1.57" upper="1.57" effort="30.0" velocity="10.0"/>
-    </joint>
-    <!-- Gripper -->
-    <link name="gripper_base">
-        <xacro:box_inertia m="0.500" l="${2*0.1}" w="${2*0.1}" h="${2*0.1}"
-                            xyz="0 0 -0.60" rpy="0 0 0" />
-        <visual>
-            <origin xyz="0 0 -0.60" rpy="0 0 0"/>
-            <geometry>
-                <mesh filename="package://aura_description/meshes/gripper_base.stl" scale="0.001 0.001 0.001"/>
-            </geometry>
-            <material name="silver"/>
-        </visual>
-        <collision>
-            <origin xyz="0 0 -0.60" rpy="0 0 0"/>
-            <geometry>
-                <mesh filename="package://aura_description/meshes/gripper_base.stl" scale="0.001 0.001 0.001"/>
-            </geometry>
-        </collision>
-    </link>
-    <joint name ="joint_5" type="revolute">
-        <parent link="claw_support"/>
-        <child link = "gripper_base"/>
-        <origin xyz="0 0 0.04" rpy="0 0 0"/>
-        <axis xyz="0 0 1"/>
-        <limit lower="-1.57" upper="1.57"
-                effort="30.0" velocity="10.0"/>
-    </joint>
-    <link name="gripper_right">
-        <xacro:box_inertia m="0.100" l="${2*0.1}" w="${2*0.1}" h="${2*0.1}"
-                            xyz="0 0.015 -0.66" rpy="0 0 0" />
-        <visual>
-            <origin xyz="0 0.015 -0.66" rpy="0 0 0"/>
-            <geometry>
-                <mesh filename="package://aura_description/meshes/gripper_right.stl" scale="0.001 0.001 0.001"/>
-            </geometry>
-            <material name="silver"/>
-        </visual>
-        <collision>
-            <origin xyz="0 0.015 -0.66" rpy="0 0 0"/>
-            <geometry>
-                <mesh filename="package://aura_description/meshes/gripper_right.stl" scale="0.001 0.001 0.001"/>
-            </geometry>
-        </collision>
-    </link>
-    <joint name ="joint_6" type="revolute">
-        <parent link="gripper_base"/>
-        <child link = "gripper_right"/>
-        <origin xyz="0 -0.015 0.07" rpy="0 0 0"/>
-        <axis xyz="1 0 0"/>
-        <limit lower="-0.550" upper="0"
-                effort="30.0" velocity="10.0"/>
-    </joint>
-    <link name="gripper_left">
-        <xacro:box_inertia m="0.100" l="${2*0.1}" w="${2*0.1}" h="${2*0.1}"
-                            xyz="0 -0.015 -0.66" rpy="0 0 0" />
-        <visual>
-            <origin xyz="0 -0.015 -0.66" rpy="0 0 0"/>
-            <geometry>
-                <mesh filename="package://aura_description/meshes/gripper_left.stl" scale="0.001 0.001 0.001"/>
-            </geometry>
-            <material name="silver"/>
-        </visual>
-        <collision>
-            <origin xyz="0 -0.015 -0.66" rpy="0 0 0"/>
-            <geometry>
-                <mesh filename="package://aura_description/meshes/gripper_left.stl" scale="0.001 0.001 0.001"/>
-            </geometry>
-        </collision>
-    </link>
-    <joint name ="joint_7" type="revolute">
-        <parent link="gripper_base"/>
-        <child link = "gripper_left"/>
-        <origin xyz="0 0.015 0.07" rpy="0 0 0"/>
-        <axis xyz="1 0 0"/>
-        <limit lower="0" upper="0.550"
-                effort="30.0" velocity="10.0"/>
-        <mimic joint="joint_6" multiplier="-1"/>
-    </joint>
-</robot>
+/home/utk/aura_ws/src/aura_description/urdf/aura_arm.xacro

File: install/aura_description/share/aura_description/urdf/aura_base.xacro (robot description, xacro)
@@ -1,265 +1 @@
-<?xml version="1.0" ?>
-<robot name="aura" xmlns:xacro="http://www.ros.org/wiki/xacro">
-  <xacro:arg name="is_ignition" default="true"/>
-  <xacro:arg name="is_sim" default="true"/>
-  <link name="base_footprint" />
-  <link name="base_link">
-    <inertial>
-      <origin xyz="2.6242213294725585e-17 -2.256459952565477e-17 0.016499999999999983" rpy="0 0 0"/>
-      <mass value="1.743512867727987"/>
-      <inertia ixx="0.009262" iyy="0.011957" izz="0.021216" ixy="-0.0" iyz="-0.0" ixz="-0.0"/>
-    </inertial>
-    <visual>
-      <origin xyz="0 0 0" rpy="0 0 0"/>
-      <geometry>
-        <mesh filename="package://aura_description/meshes/base_link.stl" scale="0.001 0.001 0.001"/>
-      </geometry>
-      <material name="matte_brown"/>
-    </visual>
-    <collision>
-      <origin xyz="0 0 0" rpy="0 0 0"/>
-      <geometry>
-        <mesh filename="package://aura_description/meshes/base_link.stl" scale="0.001 0.001 0.001"/>
-      </geometry>
-    </collision>
-  </link>
-  <joint name="base_footprint_joint" type="fixed">
-    <origin xyz="0.0 0.0 0.0" rpy="0.0 0.0 0.0"/>
-    <parent link="base_footprint"/>
-    <child link="base_link"/>
-  </joint>
-  <link name="wall">
-    <inertial>
-      <origin xyz="0.0 0.0 -0.033" rpy="0 0 0"/>
-      <mass value="2.7033358833743404"/>
-      <inertia ixx="0.033022" iyy="0.047623" izz="0.078083" ixy="0.0" iyz="-0.0" ixz="-0.0"/>
-    </inertial>
-    <visual>
-      <origin xyz="0.0 0.0 -0.033" rpy="0 0 0"/>
-      <geometry>
-        <mesh filename="package://aura_description/meshes/wall.stl" scale="0.001 0.001 0.001"/>
-      </geometry>
-      <material name="mud_yellow"/>
-    </visual>
-    <collision>
-      <origin xyz="0.0 0.0 -0.033" rpy="0 0 0"/>
-      <geometry>
-        <mesh filename="package://aura_description/meshes/wall.stl" scale="0.001 0.001 0.001"/>
-      </geometry>
-    </collision>
-  </link>
-  <joint name="base_wall_joint" type="fixed">
-    <origin xyz="0.0 0.0 0.033" rpy="0 0 0"/>
-    <parent link="base_link"/>
-    <child link="wall"/>
-  </joint>
-  <link name="back_castor">
-    <inertial>
-      <origin xyz="0.12 0.0 -0.015" rpy="0 0 0"/>
-      <mass value="0.030997748883593468"/>
-      <inertia ixx="3e-06" iyy="3e-06" izz="5e-06" ixy="-0.0" iyz="0.0" ixz="-0.0"/>
-    </inertial>
-    <visual>
-      <origin xyz="0.12 0.0 -0.015" rpy="0 0 0"/>
-      <geometry>
-        <mesh filename="package://aura_description/meshes/back_castor.stl" scale="0.001 0.001 0.001"/>
-      </geometry>
-      <material name="silver"/>
-    </visual>
-    <collision>
-      <origin xyz="0.0 0.0 0.0" rpy="0.0 0.0 0.0"/>
-      <geometry>
-        <sphere radius="0.015"/>
-      </geometry>
-    </collision>
-  </link>
-  <joint name="back_castor_joint" type="fixed">
-    <origin xyz="-0.12 0.0 0.0151" rpy="0 0 0"/>
-    <parent link="base_link"/>
-    <child link="back_castor"/>
-  </joint>
-  <link name="front_castor">
-    <inertial>
-      <origin xyz="-0.12 0.0 -0.15" rpy="0 0 0"/>
-      <mass value="0.030997748883593468"/>
-      <inertia ixx="3e-06" iyy="3e-06" izz="5e-06" ixy="-0.0" iyz="0.0" ixz="0.0"/>
-    </inertial>
-    <visual>
-     <origin xyz="-0.12 0.0 -0.015" rpy="0 0 0"/>
-      <geometry>
-        <mesh filename="package://aura_description/meshes/front_castor.stl" scale="0.001 0.001 0.001"/>
-      </geometry>
-      <material name="silver"/>
-    </visual>
-    <collision>
-     <!-- <origin xyz="-0.12 0.0 -0.015" rpy="0 0 0"/> -->
-     <origin xyz="0.0 0.0 0.0" rpy="0.0 0.0 0.0"/>
-      <geometry>
-        <sphere radius="0.015"/>
-      </geometry>
-    </collision>
-  </link>
-  <joint name="front_castor_joint" type="fixed">
-    <origin xyz="0.12 0.0 0.0151" rpy="0 0 0"/>
-    <parent link="base_link"/>
-    <child link="front_castor"/>
-  </joint>
-  <link name="right_wheel">
-    <inertial>
-      <origin xyz="-4.135866654458078e-07 -0.022655023372287864 -6.624769580132472e-08" rpy="0 0 0"/>
-      <mass value="2.2063738184473554"/>
-      <inertia ixx="0.00143" iyy="0.002082" izz="0.00143" ixy="0.0" iyz="-0.0" ixz="-0.0"/>
-    </inertial>
-    <visual>
-      <origin xyz="8.9e-05 0.128 -0.043091" rpy="0 0 0"/>
-      <geometry>
-        <mesh filename="package://aura_description/meshes/right_wheel.stl" scale="0.001 0.001 0.001"/>
-      </geometry>
-      <material name="cream"/>
-    </visual>
-    <collision>
-      <origin xyz="8.9e-05 0.128 -0.043091" rpy="0 0 0"/>
-      <geometry>
-        <mesh filename="package://aura_description/meshes/right_wheel.stl" scale="0.001 0.001 0.001"/>
-      </geometry>
-    </collision>
-  </link>
-  <joint name="right_wheel_joint" type="continuous">
-    <origin xyz="-8.9e-05 -0.128 0.010091" rpy="0 0 0"/>
-    <parent link="wall"/>
-    <child link="right_wheel"/>
-    <axis xyz="-0.0 1.0 0.0"/>
-  </joint>
-  <link name="left_wheel">
-    <inertial>
-      <origin xyz="-4.135866654458078e-07 0.022655023372287864 -6.624769580132472e-08" rpy="0 0 0"/>
-      <mass value="2.2063738184473554"/>
-      <inertia ixx="0.00143" iyy="0.002082" izz="0.00143" ixy="0.0" iyz="-0.0" ixz="-0.0"/>
-    </inertial>
-    <visual>
-      <origin xyz="8.9e-05 -0.128 -0.043091" rpy="0 0 0"/>
-      <geometry>
-        <mesh filename="package://aura_description/meshes/left_wheel.stl" scale="0.001 0.001 0.001"/>
-      </geometry>
-      <material name="cream"/>
-    </visual>
-    <collision>
-      <origin xyz="8.9e-05 -0.128 -0.043091" rpy="0 0 0"/>
-      <geometry>
-        <mesh filename="package://aura_description/meshes/left_wheel.stl" scale="0.001 0.001 0.001"/>
-      </geometry>
-    </collision>
-  </link>
-  <joint name="left_wheel_joint" type="continuous">
-    <origin xyz="-8.9e-05 0.128 0.010091" rpy="0 0 0"/>
-    <parent link="wall"/>
-    <child link="left_wheel"/>
-    <axis xyz="0.0 1.0 -0.0"/>
-  </joint>
-  <link name="imu_link">
-    <inertial>
-      <origin xyz="0.0 0.0 -0.033" rpy="0 0 0"/>
-      <mass value="0.011338921279200002"/>
-      <inertia ixx="1e-06" iyy="1e-06" izz="2e-06" ixy="-0.0" iyz="-0.0" ixz="-0.0"/>
-    </inertial>
-    <visual>
-      <origin xyz="0.0 0.0 -0.033" rpy="0 0 0"/>
-      <geometry>
-        <mesh filename="package://aura_description/meshes/imu.stl" scale="0.001 0.001 0.001"/>
-      </geometry>
-      <material name="purple"/>
-    </visual>
-    <collision>
-      <origin xyz="0.0 0.0 -0.033" rpy="0 0 0"/>
-      <geometry>
-        <mesh filename="package://aura_description/meshes/imu.stl" scale="0.001 0.001 0.001"/>
-      </geometry>
-    </collision>
-  </link>
-  <joint name="base_imu_joint" type="fixed">
-    <origin xyz="0.0 0.0 0.033" rpy="0 0 0"/>
-    <parent link="base_link"/>
-    <child link="imu_link"/>
-  </joint>
-  <link name="top_plate">
-    <inertial>
-      <origin xyz="0.0 0.0 -0.1" rpy="0 0 0"/>
-      <mass value="2.036265014260499"/>
-      <inertia ixx="0.005548" iyy="0.007098" izz="0.01187" ixy="0.0" iyz="-0.0" ixz="-0.000137"/>
-    </inertial>
-    <visual>
-      <origin xyz="0.0 0.0 -0.1" rpy="0 0 0"/>
-      <geometry>
-        <mesh filename="package://aura_description/meshes/top_plate.stl" scale="0.001 0.001 0.001"/>
-      </geometry>
-      <material name="matte_brown"/>
-    </visual>
-    <collision>
-      <origin xyz="0.0 0.0 -0.1" rpy="0 0 0"/>
-      <geometry>
-        <mesh filename="package://aura_description/meshes/top_plate.stl" scale="0.001 0.001 0.001"/>
-      </geometry>
-    </collision>
-  </link>
-  <joint name="base_top_plate_joint" type="fixed">
-    <origin xyz="0.0 0.0 0.1" rpy="0 0 0"/>
-    <parent link="base_link"/>
-    <child link="top_plate"/>
-  </joint>
-  <link name="camera_link">
-    <inertial>
-     <origin xyz="-0.15 0.0 -0.118" rpy="0 0 0"/>
-      <mass value="0.29820209775649525"/>
-      <inertia ixx="0.000242" iyy="2.3e-05" izz="0.000242" ixy="0.0" iyz="0.0" ixz="-0.0"/>
-    </inertial>
-    <visual>
-      <origin xyz="-0.15 0.0 -0.118" rpy="0 0 0"/>
-      <geometry>
-        <mesh filename="package://aura_description/meshes/camera.stl" scale="0.001 0.001 0.001"/>
-      </geometry>
-      <material name="silver"/>
-    </visual>
-    <collision>
-      <origin xyz="-0.15 0.0 -0.118" rpy="0 0 0"/>
-      <geometry>
-        <mesh filename="package://aura_description/meshes/camera.stl" scale="0.001 0.001 0.001"/>
-      </geometry>
-    </collision>
-  </link>
-  <joint name="base_camera_joint" type="fixed">
-    <origin xyz="0.15 0.0 0.118" rpy="0 0 0"/>
-    <parent link="base_link"/>
-    <child link="camera_link"/>
-  </joint>
-    <link name="camera_link_optical" />
-    <joint name="camera_optical_joint" type="fixed">
-        <parent link="camera_link"/>
-        <child link="camera_link_optical"/>
-        <origin xyz="0 0 0" rpy="${-pi/2} 0 ${-pi/2}"/>
-    </joint>
-  <link name="lidar_link">
-    <inertial>
-      <origin xyz="0.0 0.0 -0.16" rpy="0 0 0"/>
-      <mass value="0.5574542584878225"/>
-      <inertia ixx="0.000238" iyy="0.000472" izz="0.000552" ixy="-5e-06" iyz="-2e-06" ixz="-4.7e-05"/>
-    </inertial>
-    <visual>
-      <origin xyz="0.0 0.0 -0.16" rpy="0 0 0"/>
-      <geometry>
-        <mesh filename="package://aura_description/meshes/lidar.stl" scale="0.001 0.001 0.001"/>
-      </geometry>
-      <material name="silver"/>
-    </visual>
-    <collision>
-      <origin xyz="0.0 0.0 -0.16" rpy="0 0 0"/>
-      <geometry>
-        <mesh filename="package://aura_description/meshes/lidar.stl" scale="0.001 0.001 0.001"/>
-      </geometry>
-    </collision>
-  </link>
-  <joint name="base_lidar_joint" type="fixed">
-    <origin xyz="0.0 0.0 0.16" rpy="0 0 0"/>
-    <parent link="base_link"/>
-    <child link="lidar_link"/>
-  </joint>
-</robot>
+/home/utk/aura_ws/src/aura_description/urdf/aura_base.xacro
