Commit message: Both Color Bars Woking and Auto Docking

File: install/aura_description/share/aura_description/urdf/aura_gazebo.xacro (robot description, xacro)
@@ -1,154 +1 @@
-<?xml version="1.0" ?>
-<robot name="aura" xmlns:xacro="http://www.ros.org/wiki/xacro" >
-    <!-- Aura Wheels -->
-    <gazebo reference="back_castor">
-        <mu1>0.1</mu1>
-        <mu2>0.1</mu2>
-        <kp>1000000.0</kp>
-        <kd>100.0</kd>
-        <minDepth>0.001</minDepth>
-        <maxVel>1.0</maxVel>
-    </gazebo>
-    <gazebo reference="front_castor">
-        <mu1>0.1</mu1>
-        <mu2>0.1</mu2>
-        <kp>1000000.0</kp>
-        <kd>100.0</kd>
-        <minDepth>0.001</minDepth>
-        <maxVel>1.0</maxVel>
-    </gazebo>
-    <gazebo reference="right_wheel">
-        <mu1>1000000000000000.0</mu1>
-        <mu2>1000000000000000.0</mu2>
-        <kp>1000000000000.0</kp>
-        <kd>10.0</kd>
-        <minDepth>0.001</minDepth>
-        <maxVel>0.1</maxVel>
-        <fdir1>1 0 0</fdir1>
-    </gazebo>
-    <gazebo reference="left_wheel">
-        <mu1>1000000000000000.0</mu1>
-        <mu2>1000000000000000.0</mu2>
-        <kp>1000000000000.0</kp>
-        <kd>10.0</kd>
-        <minDepth>0.001</minDepth>
-        <maxVel>0.1</maxVel>
-        <fdir1>1 0 0</fdir1>
-    </gazebo>
-    <!-- ROS 2 Control -->
-    <gazebo>
-        <!-- ROS 2 Humble -->
-        <plugin filename="ign_ros2_control-system" name="ign_ros2_control::IgnitionROS2ControlPlugin">
-            <parameters>$(find aura_controller)/config/aura_controllers.yaml</parameters>
-        </plugin>
-        <plugin filename="ignition-gazebo-imu-system" name="ignition::gazebo::systems::Imu">
-        </plugin>
-        <plugin filename="ignition-gazebo-sensors-system" name="ignition::gazebo::systems::Sensors">
-            <render_engine>ogre2</render_engine>
-        </plugin>
-    </gazebo>
-    <!-- Aura Sensors -->
-    <gazebo reference="imu_link">
-        <sensor name="imu" type="imu">
-            <always_on>true</always_on>
-            <update_rate>100</update_rate>
-            <gz_frame_id>imu_link</gz_frame_id>
-            <topic>imu</topic>
-            <imu>
-                <angular_velocity>
-                    <x>
-                        <noise type="gaussian">
-                            <mean>0.0</mean>
-                            <stddev>2e-4</stddev>
-                        </noise>
-                    </x>
-                    <y>
-                        <noise type="gaussian">
-                            <mean>0.0</mean>
-                            <stddev>2e-4</stddev>
-                        </noise>
-                    </y>
-                    <z>
-                        <noise type="gaussian">
-                            <mean>0.0</mean>
-                            <stddev>2e-4</stddev>
-                        </noise>
-                    </z>
-                </angular_velocity>
-                <linear_acceleration>
-                    <x>
-                        <noise type="gaussian">
-                            <mean>0.0</mean>
-                            <stddev>1.7e-2</stddev>
-                        </noise>
-                    </x>
-                    <y>
-                        <noise type="gaussian">
-                            <mean>0.0</mean>
-                            <stddev>1.7e-2</stddev>
-                        </noise>
-                    </y>
-                    <z>
-                        <noise type="gaussian">
-                            <mean>0.0</mean>
-                            <stddev>1.7e-2</stddev>
-                        </noise>
-                    </z>
-                </linear_acceleration>
-            </imu>
-        </sensor>
-    </gazebo>
-    <gazebo reference="lidar_link">
-        <sensor name="lidar" type="gpu_lidar">
-            <pose>0 0 0 0 0 0</pose>
-            <always_on>true</always_on>
-            <visualize>true</visualize>
-            <topic>scan</topic>
-            <update_rate>5</update_rate>
-            <gz_frame_id>lidar_link</gz_frame_id>
-            <lidar>
-                <scan>
-                    <horizontal>
-                        <samples>360</samples>
-                        <resolution>1.00000</resolution>
-                        <min_angle>0.000000</min_angle>
-                        <max_angle>6.280000</max_angle>
-                    </horizontal>
-                </scan>
-                <range>
-                    <min>0.120000</min>
-                    <max>12.0</max>
-                    <resolution>0.02</resolution>
-                </range>
-                <noise>
-                    <type>gaussian</type>
-                    <mean>0.0</mean>
-                    <stddev>0.01</stddev>
-                </noise>
-            </lidar>
-        </sensor>
-    </gazebo>
-    <gazebo reference="camera_link">
-        <sensor name="camera" type="camera">
-            <pose>0 0 0 0 0 0 </pose>
-            <visualize>true</visualize>
-            <update_rate>10.0</update_rate>
-            <alwaysOn>true</alwaysOn>
-            <topic>camera/image_raw</topic>
-            <gz_frame_id>camera_link_optical</gz_frame_id>
-            <camera name="intel_realsense_r200">
-                <camera_info_topic>camera/camera_info</camera_info_topic>
-                <horizontal_fov>1.3962634</horizontal_fov>
-                <image>
-                    <width>640</width>
-                    <height>480</height>
-                    <format>R8G8B8</format>
-                </image>
-                <clip>
-                    <near>0.05</near>
-                    <far>8.0</far>
-                </clip>
-            </camera>
-        </sensor>
-  </gazebo>
-</robot>
+/home/utk/aura_ws/src/aura_description/urdf/aura_gazebo.xacro

File: install/aura_description/share/aura_description/urdf/aura_materials.xacro (robot description, xacro)
@@ -1,60 +1 @@
-<?xml version="1.0" ?>
-<robot name="aura" xmlns:xacro="http://www.ros.org/wiki/xacro">
-    <!-- Rviz Materials -->
-    <!-- Silver material -->
-    <material name="silver">
-        <color rgba="0.700 0.700 0.700 1.000"/>
-    </material>
-    <!-- Mud Yellow -->
-    <material name="mud_yellow">
-        <color rgba="0.804 0.522 0.247 1.000"/>
-    </material>
-    <!-- Purple -->
-    <material name="purple">
-        <color rgba="0.502 0.000 0.502 1.000"/>
-    </material>
-    <!-- Matte Brown -->
-    <material name="matte_brown">
-        <color rgba="0.545 0.271 0.075 1.000"/> <!-- RGB for a rich matte brown -->
-    </material>
-    <!-- Cream -->
-    <material name="cream">
-        <color rgba="1.000 0.980 0.850 1.000"/>
-    </material>
-    <xacro:macro name="box_inertia" params="m l w h xyz rpy">
-        <inertial>
-            <origin xyz="${xyz}" rpy="${rpy}" />
-            <mass value="${m}" />
-            <inertia ixx="${(m/12) * (h*h + l*l)}" ixy="0" ixz="0"
-                     iyy="${(m/12) * (w*w + l*l)}" iyz="0"
-                     izz="${(m/12) * (w*w + h*h)}" />
-        </inertial>
-    </xacro:macro>
-    <xacro:macro name="cylinder_inertia" params="m r h xyz rpy">
-        <inertial>
-            <origin xyz="${xyz}" rpy="${rpy}" />
-            <mass value="${m}" />
-            <inertia ixx="${(m/12) * (3*r*r + h*h)}" ixy="0" ixz="0"
-                     iyy="${(m/12) * (3*r*r + h*h)}" iyz="0"
-                     izz="${(m/2) * (r*r)}" />
-        </inertial>
-    </xacro:macro>
-    <!-- <xacro:macro name="sphere_inertia" params="m r xyz rpy">
-        <inertial>
-            <origin xyz="${xyz}" rpy="${rpy}" />
-            <mass value="${m}" />
-            <inertia ixx="${((2*m)/5) * (r*r)}" ixy="0" ixz="0"
-                     iyy="${((2*m)/5) * (r*r)}" iyz="0"
-                     izz="${((2*m)/5) * (r*r)}" />
-        </inertial>
-    </xacro:macro> -->
-    <xacro:macro name="default_inertial" params="mass">
-        <inertial>
-            <origin xyz="0 0 0" rpy="0 0 0"/>
-            <mass value="${mass}" />
-            <inertia ixx="1.0" ixy="0.0" ixz="0.0"
-                     iyy="1.0" iyz="0.0"
-                     izz="1.0" />
-        </inertial>
-    </xacro:macro>
-</robot>
+/home/utk/aura_ws/src/aura_description/urdf/aura_materials.xacro

File: install/aura_description/share/aura_description/urdf/aura_ros2control.xacro (robot description, xacro)
@@ -1,91 +1 @@
-<?xml version="1.0"?>
-<robot name="aura" xmlns:xacro="http://www.ros.org/wiki/xacro">
-    <ros2_control name="RobotSystem" type="system">
-        <xacro:property name="PI" value="3.14159265359" />
-        <!-- ros2_control Gazebo -->
-        <xacro:if value="$(arg is_sim)">
-            <!-- ROS 2 Humble -->
-            <xacro:if value="$(arg is_ignition)">
-                <hardware>
-                    <plugin>ign_ros2_control/IgnitionSystem</plugin>
-                </hardware>
-            </xacro:if>
-            <!-- ROS 2 Iron or above -->
-            <xacro:unless value="$(arg is_ignition)">
-                <hardware>
-                    <plugin>gz_ros2_control/GazeboSimSystem</plugin>
-                </hardware>
-            </xacro:unless>
-            <joint name="joint_7">
-                <param name="mimic">joint_6</param>
-                <param name="multiplier">-1</param>
-            </joint>
-        </xacro:if>
-        <!-- ros2_control Real Robot -->
-        <xacro:unless value="$(arg is_sim)">
-            <hardware>
-                <plugin>aura_firmware/auraInterface</plugin>
-                <param name="port">/dev/ttyUSB0</param>
-            </hardware>
-        </xacro:unless>
-        <!-- ros2_control Common Interfaces -->
-        <joint name="right_wheel_joint">
-            <command_interface name="velocity">
-              <param name="min">-1</param>
-              <param name="max">1</param>
-            </command_interface>
-            <state_interface name="position" />
-            <state_interface name="velocity" />
-        </joint>
-        <joint name="left_wheel_joint">
-            <command_interface name="velocity">
-              <param name="min">-1</param>
-              <param name="max">1</param>
-            </command_interface>
-            <state_interface name="position" />
-            <state_interface name="velocity" />
-        </joint>
-        <joint name="joint_1">
-            <command_interface name="position">
-            <param name="min">-${PI / 2}</param>
-            <param name="max">${PI / 2}</param>
-            </command_interface>
-            <state_interface name="position"/>
-        </joint>
-        <joint name="joint_2">
-            <command_interface name="position">
-            <param name="min">-${PI / 2}</param>
-            <param name="max">${PI / 2}</param>
-            </command_interface>
-            <state_interface name="position"/>
-        </joint>
-        <joint name="joint_3">
-            <command_interface name="position">
-            <param name="min">-${PI / 2}</param>
-            <param name="max">${PI / 2}</param>
-            </command_interface>
-            <state_interface name="position"/>
-        </joint>
-        <joint name="joint_4">
-            <command_interface name="position">
-            <param name="min">-${PI / 2}</param>
-            <param name="max">${PI / 2}</param>
-            </command_interface>
-            <state_interface name="position"/>
-        </joint>
-        <joint name="joint_5">
-            <command_interface name="position">
-            <param name="min">-${PI / 2}</param>
-            <param name="max">${PI / 2}</param>
-            </command_interface>
-            <state_interface name="position"/>
-        </joint>
-        <joint name="joint_6">
-            <command_interface name="position">
-            <param name="min">-0.550</param>
-            <param name="max">0.0</param>
-            </command_interface>
-            <state_interface name="position"/>
-        </joint>
-    </ros2_control>
-</robot>
+/home/utk/aura_ws/src/aura_description/urdf/aura_ros2control.xacro
